Commit message: Added the velocity controller and caddy POC testing environment.

File: caddy_poc/uwsim_lv/data/scenes/diver.urdf (robot description, URDF)
Before this commit: robot platforma, 1 links, 0 joints
Links:
- link base_link: geometry visual mesh filename=package://uwsim_lv/data/robots/diver/diver.osg

File: caddy_poc/uwsim_lv/data/scenes/pladypos.urdf (robot description, URDF)
Before this commit: robot platforma, 1 links, 0 joints
Links:
- link base_link: geometry visual mesh filename=package://uwsim_lv/data/robots/pladypos/pladypos.osg
