Commit message: Added the navcon2udp for labview simulations and updated the urdf models.

File: caddy_uwsim/data/scenes/diver.urdf (robot description, URDF)
Before this commit: robot diver, 1 links, 0 joints
Links:
- link base_link: geometry visual mesh filename=package://caddy_uwsim/data/robots/diver/diver.osg

File: caddy_uwsim/data/scenes/pladypos.urdf (robot description, URDF)
Before this commit: robot pladypos, 1 links, 0 joints
Links:
- link base_link: geometry visual mesh filename=package://caddy_uwsim/data/robots/pladypos/pladypos.osg

Commit message: Updated model download scripts.

File: caddy_uwsim/data/scenes/diver.urdf (robot description, URDF)
Before this commit: robot diver, 1 links, 0 joints
Links:
- link base_link: geometry visual mesh filename=package://caddy_uwsim/data/robots/diver/diver.3ds
