Commit message: Changed the model node to generate GPS and IMU simulation data. Added the USBL nodelets for testing. Introduced the transform frames to be used with the TF library. Started working on the velocity control improvements.

File: cart2/data/scenes/cart2.urdf (robot description, URDF)
Before this commit: robot cart2, 1 links, 0 joints
Links:
- link base_link: geometry visual mesh filename=package://cart2/data/robots/cart2.wrl
